File: hardware/kicad/6502/6502.kicad_pcb (KiCad board)
At the start: 2 copper layers, 172.4 x 131.3 mm, 47 parts, among them J1 Barrel_Jack, J2 Bus_Header, J3 LCD_Header, J4 UART_Header, J5 VIA_Header, SW1 SW_Push, SW2 SW_Push, SW3 SW_Push, SW4 SW_Push, SW5 SW_Push, U1 L7805, U2 W65C02SxP, U3 28C256, U4 HM62256BLP, U5 W65C22SxP, U6 74LS00, U7 74LS00, U8 W65C51NxP, U9 74LS00, X1 TFT680, X2 TFT680

Commit message: Added VGA testing components.
Parts:
- removed the C2 at (103.3, 72.2)
- removed the C7 at (93.9, 99.9)
- added C13: 0.1µF, Capacitor_THT:C_Disc_D5.0mm_W2.5mm_P2.50mm, F.Cu at (327.8, 142.6)
- added C14: 0.1µF, Capacitor_THT:C_Disc_D5.0mm_W2.5mm_P2.50mm, F.Cu at (327.7, 69.9)
- added C15: 0.1µF, Capacitor_THT:C_Disc_D5.0mm_W2.5mm_P2.50mm, F.Cu at (279.0, 69.9)
- added C16: 0.1µF, Capacitor_THT:C_Disc_D5.0mm_W2.5mm_P2.50mm, F.Cu at (311.3, 107.2)
- added C17: 0.1µF, Capacitor_THT:C_Disc_D5.0mm_W2.5mm_P2.50mm, F.Cu at (262.3, 107.2)
- added C18: 0.1µF, Capacitor_THT:C_Disc_D5.0mm_W2.5mm_P2.50mm, F.Cu at (311.5, 69.9)
- added C19: 0.1µF, Capacitor_THT:C_Disc_D5.0mm_W2.5mm_P2.50mm, F.Cu at (132.2, 131.2)
- added C20: 0.1µF, Capacitor_THT:C_Disc_D5.0mm_W2.5mm_P2.50mm, F.Cu at (327.5, 107.2)
- added C21: 0.1µF, Capacitor_THT:C_Disc_D5.0mm_W2.5mm_P2.50mm, F.Cu at (295.3, 142.6)
- added C22: 0.1µF, Capacitor_THT:C_Disc_D5.0mm_W2.5mm_P2.50mm, F.Cu at (279.0, 142.6)
- added C23: 0.1µF, Capacitor_THT:C_Disc_D5.0mm_W2.5mm_P2.50mm, F.Cu at (262.6, 69.9)
- added C9: 0.1µF, Capacitor_THT:C_Disc_D5.0mm_W2.5mm_P2.50mm, F.Cu at (154.8, 101.1)
- added J10: VGA_Data_Header, Connector_PinHeader_2.54mm:PinHeader_2x08_P2.54mm_Vertical, F.Cu at (243.1, 166.0)
- added J6: VGA_Out, VGA:TE_1-1734530-1, F.Cu at (161.1, 76.3)
- added J7: GAL_Header, Connector_PinSocket_2.54mm:PinSocket_1x16_P2.54mm_Vertical, F.Cu at (218.1, 190.2)
- added J8: VGA_Address_Header, Connector_PinHeader_2.54mm:PinHeader_2x20_P2.54mm_Vertical, F.Cu at (331.2, 190.1)
- added J9: VGA_Clock, Connector_PinHeader_2.54mm:PinHeader_2x03_P2.54mm_Vertical, F.Cu at (112.5, 98.4)
- added R10: 1.5k, Resistor_THT:R_Axial_DIN0207_L6.3mm_D2.5mm_P10.16mm_Horizontal, F.Cu at (195.1, 84.3)
- added R11: 680Ω, Resistor_THT:R_Axial_DIN0207_L6.3mm_D2.5mm_P10.16mm_Horizontal, F.Cu at (195.1, 67.9)
- added R12: 1.5k, Resistor_THT:R_Axial_DIN0207_L6.3mm_D2.5mm_P10.16mm_Horizontal, F.Cu at (195.1, 71.2)
- added R13: 1k, Resistor_THT:R_Axial_DIN0207_L6.3mm_D2.5mm_P10.16mm_Horizontal, F.Cu at (265.4, 142.4)
- added R14: 1k, Resistor_THT:R_Axial_DIN0207_L6.3mm_D2.5mm_P10.16mm_Horizontal, F.Cu at (262.0, 142.4)
- added R15: 1k, Resistor_THT:R_Axial_DIN0207_L6.3mm_D2.5mm_P10.16mm_Horizontal, F.Cu at (258.7, 142.4)
- added R16: 1k, Resistor_THT:R_Axial_DIN0207_L6.3mm_D2.5mm_P10.16mm_Horizontal, F.Cu at (255.4, 142.4)
- added R7: 680Ω, Resistor_THT:R_Axial_DIN0207_L6.3mm_D2.5mm_P10.16mm_Horizontal, F.Cu at (195.1, 74.4)
- added R8: 1.5k, Resistor_THT:R_Axial_DIN0207_L6.3mm_D2.5mm_P10.16mm_Horizontal, F.Cu at (185.0, 77.7)
- added R9: 680Ω, Resistor_THT:R_Axial_DIN0207_L6.3mm_D2.5mm_P10.16mm_Horizontal, F.Cu at (195.1, 81.0)
- added SW6: SW_VGA_CLOCK, Switch:SW_THT_DPDT, F.Cu at (95.9, 99.1)
- added SW7: DMA_DIP, Button_Switch_THT:SW_DIP_SPSTx04_Slide_9.78x12.34mm_W7.62mm_P2.54mm, F.Cu at (264.2, 163.3)
- added SW8: SW_SPDT, Switch:SW_THT_DPDT, F.Cu at (95.2, 85.5)
- added U10: 74HC00, Package_DIP:DIP-14_W7.62mm_Socket, F.Cu at (322.6, 75.4)
- added U11: 74LS161, Package_DIP:DIP-16_W7.62mm_Socket, F.Cu at (257.3, 113.0)
- added U12: GAL16V8, Package_DIP:DIP-20_W7.62mm_Socket, F.Cu at (306.1, 113.0)
- added U13: 74HC00, Package_DIP:DIP-14_W7.62mm_Socket, F.Cu at (322.3, 113.0)
- added U14: 74HC74, Package_DIP:DIP-14_W7.62mm_Socket, F.Cu at (127.0, 135.7)
- added U15: 74HC245, Package_DIP:DIP-20_W7.62mm_Socket, F.Cu at (290.2, 147.9)
- added U16: 74HC245, Package_DIP:DIP-20_W7.62mm_Socket, F.Cu at (306.4, 147.9)
- added U17: 74HC245, Package_DIP:DIP-20_W7.62mm_Socket, F.Cu at (322.6, 147.9)
- added U18: 74LS161, Package_DIP:DIP-16_W7.62mm_Socket, F.Cu at (273.8, 74.8)
- added U19: 74LS161, Package_DIP:DIP-16_W7.62mm_Socket, F.Cu at (290.1, 74.8)
- added U20: 74LS161, Package_DIP:DIP-16_W7.62mm_Socket, F.Cu at (273.6, 113.0)
- added U21: 74LS161, Package_DIP:DIP-16_W7.62mm_Socket, F.Cu at (289.9, 113.0)
- added X3: TFT660, Oscillator:Oscillator_DIP-8, F.Cu at (110.5, 124.0)
- added X4: TFT680, Oscillator:Oscillator_DIP-14, F.Cu at (118.0, 149.4)
- U1: value L7805 -> GAL16V8; footprint Package_TO_SOT_THT:TO-220-3_Horizontal_TabDown -> Package_DIP:DIP-20_W7.62mm_Socket
- U6: value 74LS00 -> 74LS161; footprint Package_DIP:DIP-14_W7.62mm_Socket -> Package_DIP:DIP-16_W7.62mm_Socket
- U7, U9: value 74LS00 -> GAL16V8; footprint Package_DIP:DIP-14_W7.62mm_Socket -> Package_DIP:DIP-20_W7.62mm_Socket
- moved NW 313.2 mm to (335.2, 202.9)
- moved C7 210.0 mm to (314.0, 142.6), turned to 180 degrees
- moved U9 197.8 mm to (273.9, 147.9)
- moved U7 180.5 mm to (306.3, 75.1)
- moved C3 163.6 mm to (244.6, 98.8), turned to -90 degrees
- moved J2 162.8 mm to (273.2, 190.1), turned to -90 degrees
- moved NE 153.8 mm to (86.7, 62.0)
- moved C4 144.0 mm to (244.8, 123.1)
- moved SE 134.2 mm to (335.2, 62.1)
- moved U6 113.5 mm to (257.5, 74.8)
- moved J5 111.4 mm to (173.7, 190.1), turned to -90 degrees
- moved C8 105.9 mm to (141.7, 138.3), turned to 90 degrees
- moved C12 104.8 mm to (295.0, 107.2), turned to 0 degrees
- moved C5 85.2 mm to (244.8, 148.5)
- moved U1 85.1 mm to (160.2, 101.0), turned to 90 degrees
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- renumbered C10 to C11, C8 to C2, C9 to C3, C3 to C4, C4 to C5, C5 to C6, C6 to C7, C11 to C8
Connections:
- C1 pad 1: Net-(C1-Pad1) -> VCC
- C11 pad 1: /PHI3 -> /PHI2
- D1 pad 1: Net-(C1-Pad1) -> VCC
- J1 pad 1: Net-(D1-Pad2) -> Net-(J1-Pad1)
- J2 pad 24: unconnected-(J2-Pad24) -> /~{HBLANK}
- J2 pad 26: unconnected-(J2-Pad26) -> /~{VBLANK}
- J2 pad 28: unconnected-(J2-Pad28) -> /~{HSYNC}
- J2 pad 30: unconnected-(J2-Pad30) -> /~{VSYNC}
- J2 pad 34: /PHI2 -> /CPU_CLOCK
- J2 pad 35: /PHI2 -> /CPU_CLOCK
- J2 pad 36: /~{PHI2} -> /~{CPU_CLOCK}
- J2 pad 38: /RDY -> ~{DMA}
- U1 pad 1: Net-(C1-Pad1) -> /A12
- U1 pad 2: GND -> /A13
- U1 pad 3: VCC -> /A14
- U2 pad 2: /RDY -> ~{DMA}
- U2 pad 36: /RDY -> ~{DMA}
- U2 pad 37: /PHI2 -> /CPU_CLOCK
- U4 pad 22: /A14 -> /~{RAMOE}
- U5 pad 23: /~{VIACS2} -> /~{VIACS}
- U5 pad 24: /A13 -> VCC
- U5 pad 25: /PHI2 -> /CPU_CLOCK
- U6 pad 1: /A14 -> /VGA/Horizontal/~{H_CLR}
- U6 pad 10: /A15 -> VCC
- U6 pad 11: /~{ROMCS} -> /VGA/Horizontal/H_Q3
- U6 pad 12: /A14 -> /VGA/Horizontal/H_Q2
- U6 pad 13: /A15 -> /VGA/Horizontal/H_Q1
- U6 pad 14: VCC -> /VGA/Horizontal/H_Q0
- U6 pad 2: /A14 -> /VGA/Horizontal/VGA_CLOCK
- U6 pad 3: /~{A14} -> unconnected-(U6-Pad3)
- U6 pad 4: /A14 -> unconnected-(U6-Pad4)
- U6 pad 5: /~{A15} -> unconnected-(U6-Pad5)
- U6 pad 6: /~{VIACS2} -> unconnected-(U6-Pad6)
- U6 pad 7: GND -> VCC
- U6 pad 8: /~{A15} -> GND
- U6 pad 9: /A15 -> VCC
- U7 pad 1: /PHI2 -> /VGA/Horizontal/H_Q0
- U7 pad 10: /~{A14} -> GND
- U7 pad 11: Net-(U7-Pad11) -> /VGA/Horizontal/H_Q9
- U7 pad 12: Net-(U7-Pad12) -> /VGA/Horizontal/GAL1_O3
- U7 pad 13: /RDY -> /VGA/Horizontal/GAL1_O2
- U7 pad 14: VCC -> /VGA/Horizontal/GAL1_O1
- U7 pad 2: /PHI2 -> /VGA/Horizontal/H_Q1
- U7 pad 3: /~{PHI2} -> /VGA/Horizontal/H_Q2
- U7 pad 4: Net-(U7-Pad11) -> /VGA/Horizontal/H_Q3
- U7 pad 5: Net-(U7-Pad11) -> /VGA/Horizontal/H_Q4
- U7 pad 6: /~{RAMCS} -> /VGA/Horizontal/H_Q5
- U7 pad 7: GND -> /VGA/Horizontal/H_Q6
- U7 pad 8: Net-(U7-Pad12) -> /VGA/Horizontal/H_Q7
- U7 pad 9: /PHI2 -> /VGA/Horizontal/H_Q8
- U8 pad 2: /~{ACIACS} -> VCC
- U8 pad 27: /PHI2 -> /CPU_CLOCK
- U8 pad 3: /~{VIACS2} -> /~{ACIACS}
- U8 pad 6: /PHI3 -> /PHI2
- U9 pad 1: /A13 -> /VGA/~{HBLANK}
- U9 pad 11: unconnected-(U9-Pad11) -> /VGA/GAL3_I6
- U9 pad 12: GND -> /VGA/GAL3_O4
- U9 pad 13: GND -> /VGA/GAL3_O3
- U9 pad 14: VCC -> /VGA/GAL3_O2
- U9 pad 2: /A13 -> /VGA/~{VBLANK}
- U9 pad 3: /~{ACIACS} -> /VGA/~{CPU_CLOCK}
- U9 pad 4: GND -> /VGA/GAL3_I0
- U9 pad 5: GND -> /VGA/GAL3_I1
- U9 pad 6: unconnected-(U9-Pad6) -> /VGA/GAL3_I2
- U9 pad 7: GND -> /VGA/GAL3_I3
- U9 pad 8: unconnected-(U9-Pad8) -> /VGA/GAL3_I4
- U9 pad 9: GND -> /VGA/GAL3_I5
- X2 pad 8: /PHI3 -> /PHI2
Routing:
- net GND: track 921.7 -> 0.00 mm, vias 1 -> 0
- net /D2: track 237.1 -> 0.00 mm
- net /D1: track 221.3 -> 0.00 mm, vias 2 -> 0
- net /D0: track 219.4 -> 0.00 mm
- net /D3: track 210.0 -> 0.00 mm, vias 2 -> 0
- net /D4: track 201.3 -> 0.00 mm, vias 1 -> 0
- net /A13: track 200.3 -> 0.00 mm, vias 2 -> 0
- net /D7: track 198.3 -> 0.00 mm, vias 1 -> 0
- net /D5: track 196.6 -> 0.00 mm, vias 3 -> 0
- net /D6: track 196.2 -> 0.00 mm, vias 1 -> 0
- net /PHI2: track 187.6 -> 0.00 mm, vias 1 -> 0
- net /A14: track 178.3 -> 0.00 mm, vias 1 -> 0
- net /RDY: track 176.4 -> 0.00 mm, vias 1 -> 0
- net /A0: track 170.3 -> 0.00 mm
- net /~{RES}: track 167.6 -> 0.00 mm
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- added copper zone on B.Cu, net GND
Other:
- board size 172.4 x 131.3 mm -> 256.3 x 148.7 mm
- board text added: "1.5k"
- board text added: "1/1 Speed"
- board text added: "1/2 Speed"
- board text added: "1/4 Speed"
- board text added: "680Ω"
- board text added: "74HC74"
- board text added: "ADDRESS BUFFER 0"
- board text added: "ADDRESS BUFFER 1"
- board text added: "BA0"
- board text added: "BA1"
- board text added: "BA10"
- board text added: "BA11"
- board text added: "BA12"
- board text added: "BA13"
- board text added: "BA14"
- board text added: "BA15"
- board text added: "BA2"
- board text added: "BA3"
- board text added: "BA4"
- board text added: "BA5"
- board text added: "BA6"
- board text added: "BA7"
- board text added: "BA8"
- board text added: "BA9"
- board text added: "BD0"
- board text added: "BD1"
- board text added: "BD2"
- board text added: "BD3"
- board text added: "BD4"
- board text added: "BD5"
- board text added: "BD6"
- board text added: "BD7"
- board text added: "CPU GAL"
- board text added: "CPU_CLOCK"
- board text added: "DATA BUFFER"
- board text added: "DMA"
- board text added: "DMA PLD"
- board text added: "GAL0_01"
- board text added: "GAL0_I0"
- board text added: "GAL0_I1"
- board text added: "GAL0_I2"
- board text added: "GAL0_I3"
- board text added: "GAL0_O0"
- board text added: "GAL3_I0"
- board text added: "GAL3_I1"
- board text added: "GAL3_I2"
- board text added: "GAL3_I3"
- board text added: "GAL3_I4"
- board text added: "GAL3_I5"
- board text added: "GAL3_I6"
- board text added: "GAL3_O0"
- board text added: "GAL3_O1"
- board text added: "GAL3_O2"
- board text added: "GAL3_O3"
- board text added: "HBLANK"
- board text added: "HORIZ COUNTER 0"
- board text added: "HORIZ COUNTER 1"
- board text added: "HORIZ COUNTER 2"
- board text added: "HORIZ LATCH"
- board text added: "HORIZ PLD"
- board text added: "HSYNC"
- board text added: "H_Q0"
- board text added: "H_Q1"
- board text added: "H_Q2"
- board text added: "H_Q3"
- board text added: "H_Q4"
- board text added: "H_Q5"
- board text added: "H_Q6"
- board text added: "H_Q7"
- board text added: "H_Q8"
- board text added: "H_Q9"
- board text added: "Revision 1.2 (9/12/22)"
- board text added: "VBLANK"
- board text added: "VERTICAL COUNTER 0"
- board text added: "VERTICAL COUNTER 1"
- board text added: "VERTICAL COUNTER 2"
- board text added: "VERTICAL LATCH"
- board text added: "VERTICAL PLD"
- board text added: "VGA - HORIZONTAL"
- board text added: "VGA - OUTPUT"
- board text added: "VGA - VERTICAL"
- board text added: "VGA CLOCK 0"
- board text added: "VGA CLOCK 1"
- board text added: "VGA Clock 0 | VGA Clock 1"
- board text added: "VGA Clock Settings"
- board text added: "VGA OUT"
- board text added: "VSYNC"
- board text added: "V_Q0"
- board text added: "V_Q1"
- board text added: "V_Q2"
- board text added: "V_Q3"
- board text added: "V_Q4"
- board text added: "V_Q5"
- board text added: "V_Q6"
- board text added: "V_Q7"
- board text added: "V_Q8"
- board text added: "V_Q9"
- board text removed: "-Connect RDY to VCC W/O Graphics Card -Connect PHI1 to PHI2 W/O External Clock"
- board text removed: "74LS00"
- board text removed: "PHI2"
- board text removed: "RDY"
- board text removed: "Revision 1.1 (9/3/22)"

Commit message: Finalized revision 1.2.
Parts:
- added C10: 0.1µF, Capacitor_THT:C_Disc_D5.0mm_W2.5mm_P2.50mm, F.Cu at (295.4, 69.9)
- moved C5 53.4 mm to (278.7, 107.2), turned to 0 degrees
- moved C8 10.3 mm to (141.7, 148.6), turned to -90 degrees
- moved C7 2.42 mm to (311.6, 142.6), turned to 0 degrees
- moved C2 0.27 mm to (141.8, 112.8)
- moved SE 0.14 mm to (335.3, 62.0)
- turned C9 to 90 degrees
Connections:
- net /VGA/GAL3_I3 renamed /GAL3_I3
- net /VGA/GAL3_I4 renamed /GAL3_I4
- net /VGA/GAL3_I5 renamed /GAL3_I5
- net /VGA/GAL3_I6 renamed /GAL3_I6
- net /VGA/GAL3_O4 renamed /GAL3_O4
- J2 pad 38: ~{DMA} -> /~{DMA}
- J6 pad 13: /VGA/~{VSYNC} -> /~{VSYNC}
- J6 pad 14: /VGA/~{HSYNC} -> /~{HSYNC}
- J7 pad 10: /GAL3_O0 -> /GAL3_O1
- J7 pad 11: /GAL3_O1 -> /GAL3_O2
- J7 pad 12: /GAL3_O2 -> /GAL3_O3
- J7 pad 13: /GAL3_O3 -> VCC
- J7 pad 9: /GAL0_O1 -> /GAL3_O0
- J8 pad 10: /VGA/H_Q7 -> /H_Q7
- J8 pad 12: /VGA/H_Q8 -> /H_Q8
- J8 pad 14: /VGA/H_Q9 -> /H_Q9
- J8 pad 16: /VGA/V_Q3 -> /V_Q3
- J8 pad 18: /VGA/V_Q4 -> /V_Q4
- J8 pad 2: /VGA/H_Q3 -> /H_Q3
- J8 pad 20: /VGA/V_Q5 -> /V_Q5
- J8 pad 22: /VGA/V_Q6 -> /V_Q6
- J8 pad 24: /VGA/V_Q7 -> /V_Q7
- J8 pad 26: /VGA/V_Q8 -> /V_Q8
- J8 pad 28: /VGA/V_Q9 -> /V_Q9
- J8 pad 33: /VGA/H_Q0 -> /H_Q0
- J8 pad 34: /VGA/V_Q0 -> /V_Q0
- J8 pad 35: /VGA/H_Q1 -> /H_Q1
- J8 pad 36: /VGA/V_Q1 -> /V_Q1
- J8 pad 37: /VGA/H_Q2 -> /H_Q2
- J8 pad 38: /VGA/V_Q2 -> /V_Q2
- J8 pad 4: /VGA/H_Q4 -> /H_Q4
- J8 pad 6: /VGA/H_Q5 -> /H_Q5
- J8 pad 8: /VGA/H_Q6 -> /H_Q6
- J9 pad 2: /VGA/VGA_CLOCK -> /VGA_CLOCK
- J9 pad 4: /VGA/VGA_CLOCK -> /VGA_CLOCK
- J9 pad 6: /VGA/VGA_CLOCK -> /VGA_CLOCK
- U1 pad 1: /A12 -> /CPU_CLOCK
- U1 pad 12: /GAL0_O1 -> /GAL0_O0
- U1 pad 13: /GAL0_O0 -> /~{CPU_CLOCK}
- U1 pad 14: /~{ACIACS} -> /CPU_READY
- U1 pad 15: /~{VIACS} -> /~{ACIACS}
- U1 pad 16: /~{CPU_CLOCK} -> /~{VIACS}
- U1 pad 2: /A13 -> /A12
- U1 pad 3: /A14 -> /A13
- U1 pad 4: /A15 -> /A14
- U1 pad 5: ~{DMA} -> /A15
- U1 pad 6: /CPU_CLOCK -> /~{DMA}
- U10 pad 10: /VGA/Horizontal/~{HSYNC} -> /~{HSYNC}
- U10 pad 11: /VGA/Horizontal/~{HSYNC} -> /~{HSYNC}
- U10 pad 2: /VGA/Horizontal/~{HBLANK} -> /~{HBLANK}
- U10 pad 6: /VGA/Horizontal/~{HBLANK} -> /~{HBLANK}
- U11 pad 11: /VGA/Vertical/V_Q3 -> /V_Q3
- U11 pad 12: /VGA/Vertical/V_Q2 -> /V_Q2
- U11 pad 13: /VGA/Vertical/V_Q1 -> /V_Q1
- U11 pad 14: /VGA/Vertical/V_Q0 -> /V_Q0
- U11 pad 2: /VGA/Vertical/~{H_CLR} -> /VGA/Horizontal/~{H_CLR}
- U12 pad 1: /VGA/Vertical/V_Q0 -> /V_Q0
- U12 pad 11: /VGA/Vertical/V_Q9 -> /V_Q9
- U12 pad 2: /VGA/Vertical/V_Q1 -> /V_Q1
- U12 pad 3: /VGA/Vertical/V_Q2 -> /V_Q2
- U12 pad 4: /VGA/Vertical/V_Q3 -> /V_Q3
- U12 pad 5: /VGA/Vertical/V_Q4 -> /V_Q4
- U12 pad 6: /VGA/Vertical/V_Q5 -> /V_Q5
- U12 pad 7: /VGA/Vertical/V_Q6 -> /V_Q6
- U12 pad 8: /VGA/Vertical/V_Q7 -> /V_Q7
- U12 pad 9: /VGA/Vertical/V_Q8 -> /V_Q8
- U13 pad 10: /VGA/Vertical/~{VSYNC} -> /~{VSYNC}
- U13 pad 11: /VGA/Vertical/~{VSYNC} -> /~{VSYNC}
- U13 pad 2: /VGA/Vertical/~{VBLANK} -> /~{VBLANK}
- U13 pad 6: /VGA/Vertical/~{VBLANK} -> /~{VBLANK}
- U18 pad 11: /VGA/Horizontal/H_Q7 -> /H_Q7
- U18 pad 12: /VGA/Horizontal/H_Q6 -> /H_Q6
- U18 pad 13: /VGA/Horizontal/H_Q5 -> /H_Q5
- U18 pad 14: /VGA/Horizontal/H_Q4 -> /H_Q4
- U18 pad 2: /VGA/Horizontal/VGA_CLOCK -> /VGA_CLOCK
- U19 pad 13: /VGA/Horizontal/H_Q9 -> /H_Q9
- U19 pad 14: /VGA/Horizontal/H_Q8 -> /H_Q8
- U19 pad 2: /VGA/Horizontal/VGA_CLOCK -> /VGA_CLOCK
- U2 pad 2: ~{DMA} -> /CPU_READY
- U2 pad 36: ~{DMA} -> /CPU_READY
- U20 pad 11: /VGA/Vertical/V_Q7 -> /V_Q7
- U20 pad 12: /VGA/Vertical/V_Q6 -> /V_Q6
- U20 pad 13: /VGA/Vertical/V_Q5 -> /V_Q5
- U20 pad 14: /VGA/Vertical/V_Q4 -> /V_Q4
- U20 pad 2: /VGA/Vertical/~{H_CLR} -> /VGA/Horizontal/~{H_CLR}
- U21 pad 13: /VGA/Vertical/V_Q9 -> /V_Q9
- U21 pad 14: /VGA/Vertical/V_Q8 -> /V_Q8
- U21 pad 2: /VGA/Vertical/~{H_CLR} -> /VGA/Horizontal/~{H_CLR}
- U6 pad 11: /VGA/Horizontal/H_Q3 -> /H_Q3
- U6 pad 12: /VGA/Horizontal/H_Q2 -> /H_Q2
- U6 pad 13: /VGA/Horizontal/H_Q1 -> /H_Q1
- U6 pad 14: /VGA/Horizontal/H_Q0 -> /H_Q0
- U6 pad 2: /VGA/Horizontal/VGA_CLOCK -> /VGA_CLOCK
- U7 pad 1: /VGA/Horizontal/H_Q0 -> /H_Q0
- U7 pad 11: /VGA/Horizontal/H_Q9 -> /H_Q9
- U7 pad 2: /VGA/Horizontal/H_Q1 -> /H_Q1
- U7 pad 3: /VGA/Horizontal/H_Q2 -> /H_Q2
- U7 pad 4: /VGA/Horizontal/H_Q3 -> /H_Q3
- U7 pad 5: /VGA/Horizontal/H_Q4 -> /H_Q4
- U7 pad 6: /VGA/Horizontal/H_Q5 -> /H_Q5
- U7 pad 7: /VGA/Horizontal/H_Q6 -> /H_Q6
- U7 pad 8: /VGA/Horizontal/H_Q7 -> /H_Q7
- U7 pad 9: /VGA/Horizontal/H_Q8 -> /H_Q8
- U9 pad 1: /VGA/~{HBLANK} -> /~{CPU_CLOCK}
- U9 pad 13: /VGA/GAL3_O3 -> /GAL3_O3
- U9 pad 14: /VGA/GAL3_O2 -> /GAL3_O2
- U9 pad 15: /VGA/GAL3_O1 -> /GAL3_O1
- U9 pad 16: /VGA/GAL3_O0 -> /GAL3_O0
- U9 pad 19: /VGA/~{DMA} -> /~{DMA}
- U9 pad 2: /VGA/~{VBLANK} -> /~{HBLANK}
- U9 pad 3: /VGA/~{CPU_CLOCK} -> /~{VBLANK}
- U9 pad 4: /VGA/GAL3_I0 -> /GAL3_I0
- U9 pad 5: /VGA/GAL3_I1 -> /GAL3_I1
- U9 pad 6: /VGA/GAL3_I2 -> /GAL3_I2
Routing:
- net GND: track 0.00 -> 1259.7 mm
- net /~{HSYNC}: track 0.00 -> 371.8 mm
- net VCC: track 794.9 -> 1165.9 mm
- net /A14: track 0.00 -> 314.7 mm, vias 0 -> 1
- net /~{VSYNC}: track 0.00 -> 309.2 mm
- net /A12: track 0.00 -> 300.2 mm, vias 0 -> 2
- net /A2: track 0.00 -> 292.2 mm, vias 0 -> 1
- net /A0: track 0.00 -> 289.7 mm, vias 0 -> 1
- net /A1: track 0.00 -> 282.5 mm, vias 0 -> 1
- net /A4: track 0.00 -> 281.4 mm, vias 0 -> 3
- net /A3: track 0.00 -> 271.0 mm, vias 0 -> 2
- net /D0: track 0.00 -> 268.9 mm, vias 0 -> 1
- net /A13: track 0.00 -> 266.8 mm, vias 0 -> 2
- net /A10: track 0.00 -> 256.2 mm, vias 0 -> 1
- net /A5: track 0.00 -> 251.4 mm, vias 0 -> 1
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- removed copper zone on B.Cu, net GND
Other:
- board text added: "Revision 1.2 (9/14/22)"
- board text removed: "Revision 1.2 (9/12/22)"
