File: hardware/kicad/6502/horizontal.kicad_sch (KiCad schematic)
At the start: 5 parts, among them U10 74HC00, U18 74LS161, U19 74LS161, U6 74LS161, U7 GAL16V8

Commit message: Finalized revision 1.2.
Changed lines of the file:
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@@
+    (stroke (width 0) (type default) (color 0 0 0 0))
+  )
+  (wire (pts (xy 22.098 55.118) (xy 23.876 55.118))
     (stroke (width 0) (type default) (color 0 0 0 0))
   )
@@
     (stroke (width 0) (type default) (color 0 0 0 0))
   )
+  (wire (pts (xy 85.09 55.118) (xy 85.852 55.118))
+    (stroke (width 0) (type default) (color 0 0 0 0))
+  )
   (wire (pts (xy 85.852 55.118) (xy 85.852 53.848))
     (stroke (width 0) (type default) (color 0 0 0 0))
@@
   )
   (wire (pts (xy 52.07 42.418) (xy 57.658 42.418))
+    (stroke (width 0) (type default) (color 0 0 0 0))
+  )
+  (wire (pts (xy 144.526 54.356) (xy 147.574 54.356))
     (stroke (width 0) (type default) (color 0 0 0 0))
   )
@@
     )
     (property "Datasheet" "" (id 3) (at 101.346 74.168 0)
-      (effects (font (size 1.27 1.27)) hide)
-    )
-    (pin "1")
-  )
-  (symbol (lib_id "power:VCC") (at 85.852 55.118 90) (unit 1)
-    (in_bom yes) (on_board yes)
-    (property "Reference" "#PWR0139" (id 0) (at 89.662 55.118 0)
-      (effects (font (size 1.27 1.27)) hide)
-    )
-    (property "Value" "VCC" (id 1) (at 80.772 55.118 90))
-    (property "Footprint" "" (id 2) (at 85.852 55.118 0)
-      (effects (font (size 1.27 1.27)) hide)
-    )
-    (property "Datasheet" "" (id 3) (at 85.852 55.118 0)
       (effects (font (size 1.27 1.27)) hide)
     )
@@
     (pin "7")
   )
+  (symbol (lib_id "power:VCC") (at 85.09 55.118 90) (unit 1)
+    (in_bom yes) (on_board yes)
+    (property "Reference" "#PWR0160" (id 0) (at 88.9 55.118 0)
+      (effects (font (size 1.27 1.27)) hide)
+    )
+    (property "Value" "VCC" (id 1) (at 80.01 55.118 90))
+    (property "Footprint" "" (id 2) (at 85.09 55.118 0)
+      (effects (font (size 1.27 1.27)) hide)
+    )
+    (property "Datasheet" "" (id 3) (at 85.09 55.118 0)
+      (effects (font (size 1.27 1.27)) hide)
+    )
+    (pin "1")
+  )
+  (symbol (lib_id "power:VCC") (at 22.098 55.118 90) (unit 1)
+    (in_bom yes) (on_board yes)
+    (property "Reference" "#PWR0158" (id 0) (at 25.908 55.118 0)
+      (effects (font (size 1.27 1.27)) hide)
+    )
+    (property "Value" "VCC" (id 1) (at 17.018 55.118 90))
+    (property "Footprint" "" (id 2) (at 22.098 55.118 0)
+      (effects (font (size 1.27 1.27)) hide)
+    )
+    (property "Datasheet" "" (id 3) (at 22.098 55.118 0)
+      (effects (font (size 1.27 1.27)) hide)
+    )
+    (pin "1")
+  )
   (symbol (lib_id "74xx:74LS161") (at 163.068 53.086 0) (unit 1)
     (in_bom yes) (on_board yes) (fields_autoplaced)
@@
     (pin "8")
     (pin "9")
+  )
+  (symbol (lib_id "power:VCC") (at 144.526 54.356 90) (unit 1)
+    (in_bom yes) (on_board yes)
+    (property "Reference" "#PWR0159" (id 0) (at 148.336 54.356 0)
+      (effects (font (size 1.27 1.27)) hide)
+    )
+    (property "Value" "VCC" (id 1) (at 139.446 54.356 90))
+    (property "Footprint" "" (id 2) (at 144.526 54.356 0)
+      (effects (font (size 1.27 1.27)) hide)
+    )
+    (property "Datasheet" "" (id 3) (at 144.526 54.356 0)
+      (effects (font (size 1.27 1.27)) hide)
+    )
+    (pin "1")
   )
   (symbol (lib_id "power:VCC") (at 242.824 36.576 0) (unit 1)
@@
     (pin "7")
   )
-  (symbol (lib_id "power:VCC") (at 23.876 55.118 90) (unit 1)
-    (in_bom yes) (on_board yes)
-    (property "Reference" "#PWR0141" (id 0) (at 27.686 55.118 0)
-      (effects (font (size 1.27 1.27)) hide)
-    )
-    (property "Value" "VCC" (id 1) (at 18.796 55.118 90))
-    (property "Footprint" "" (id 2) (at 23.876 55.118 0)
-      (effects (font (size 1.27 1.27)) hide)
-    )
-    (property "Datasheet" "" (id 3) (at 23.876 55.118 0)
-      (effects (font (size 1.27 1.27)) hide)
-    )
-    (pin "1")
-  )
   (symbol (lib_id "74xx:74LS161") (at 39.37 52.578 0) (unit 1)
     (in_bom yes) (on_board yes) (fields_autoplaced)
@@
       (effects (font (size 1.27 1.27)) hide)
     )
-    (pin "1")
-  )
-  (symbol (lib_id "power:VCC") (at 147.574 54.356 90) (unit 1)
-    (in_bom yes) (on_board yes)
-    (property "Reference" "#PWR0116" (id 0) (at 151.384 54.356 0)
-      (effects (font (size 1.27 1.27)) hide)
-    )
-    (property "Value" "VCC" (id 1) (at 142.494 54.356 90))
-    (property "Footprint" "" (id 2) (at 147.574 54.356 0)
-      (effects (font (size 1.27 1.27)) hide)
-    )
-    (property "Datasheet" "" (id 3) (at 147.574 54.356 0)
-      (effects (font (size 1.27 1.27)) hide)
-    )

Commit message: BOM updates.
Parts:
- U10: ComponentPurchaseUrl (none) -> https://mou.sr/3BgiB2x; FootprintPurchaseUrl (none) -> https://mou.sr/3DAlE8i
- U18, U19, U6: ComponentPurchaseUrl (none) -> https://mou.sr/3BzZZfc; FootprintPurchaseUrl (none) -> https://mou.sr/3xt2Q7o; Purchase https://mou.sr/3BzZZfc -> (none)
- U7: ComponentPurchaseUrl (none) -> https://mou.sr/3qwJien; FootprintPurchaseUrl (none) -> https://mou.sr/3defX5i; Purchase https://mou.sr/3qwJien -> (none)
Changed lines of the file:
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@@
+      (effects (font (size 1.27 1.27)) hide)
+    )
+    (property "ComponentPurchaseUrl" "https://mou.sr/3BgiB2x" (id 4) (at 57.15 121.666 0)
+      (effects (font (size 1.27 1.27)) hide)
+    )
+    (property "FootprintPurchaseUrl" "https://mou.sr/3DAlE8i" (id 5) (at 57.15 121.666 0)
       (effects (font (size 1.27 1.27)) hide)
     )
@@
       (effects (font (size 1.27 1.27)) hide)
     )
+    (property "ComponentPurchaseUrl" "https://mou.sr/3BgiB2x" (id 4) (at 57.15 121.666 0)
+      (effects (font (size 1.27 1.27)) hide)
+    )
+    (property "FootprintPurchaseUrl" "https://mou.sr/3DAlE8i" (id 5) (at 57.15 121.666 0)
+      (effects (font (size 1.27 1.27)) hide)
+    )
     (pin "1")
     (pin "2")
@@
       (effects (font (size 1.27 1.27)) hide)
     )
-    (property "Purchase" "https://mou.sr/3BzZZfc" (id 4) (at 163.068 53.086 0)
+    (property "ComponentPurchaseUrl" "https://mou.sr/3BzZZfc" (id 4) (at 163.068 53.086 0)
+      (effects (font (size 1.27 1.27)) hide)
+    )
+    (property "FootprintPurchaseUrl" "https://mou.sr/3xt2Q7o" (id 5) (at 163.068 53.086 0)
       (effects (font (size 1.27 1.27)) hide)
     )
@@
       (effects (font (size 1.27 1.27)) hide)
     )
-    (property "Purchase" "https://mou.sr/3qwJien" (id 4) (at 242.824 54.356 0)
+    (property "ComponentPurchaseUrl" "https://mou.sr/3qwJien" (id 4) (at 242.824 54.356 0)
+      (effects (font (size 1.27 1.27)) hide)
+    )
+    (property "FootprintPurchaseUrl" "https://mou.sr/3defX5i" (id 5) (at 242.824 54.356 0)
       (effects (font (size 1.27 1.27)) hide)
     )
@@
       (effects (font (size 1.27 1.27)) hide)
     )
+    (property "ComponentPurchaseUrl" "https://mou.sr/3BgiB2x" (id 4) (at 57.15 121.666 0)
+      (effects (font (size 1.27 1.27)) hide)
+    )
+    (property "FootprintPurchaseUrl" "https://mou.sr/3DAlE8i" (id 5) (at 57.15 121.666 0)
+      (effects (font (size 1.27 1.27)) hide)
+    )
     (pin "1")
     (pin "2")
@@
       (effects (font (size 1.27 1.27)) hide)
     )
-    (property "Purchase" "https://mou.sr/3BzZZfc" (id 4) (at 101.346 53.848 0)
+    (property "ComponentPurchaseUrl" "https://mou.sr/3BzZZfc" (id 4) (at 101.346 53.848 0)
+      (effects (font (size 1.27 1.27)) hide)
+    )
+    (property "FootprintPurchaseUrl" "https://mou.sr/3xt2Q7o" (id 5) (at 101.346 53.848 0)
       (effects (font (size 1.27 1.27)) hide)
     )
@@
       (effects (font (size 1.27 1.27)) hide)
     )
+    (property "ComponentPurchaseUrl" "https://mou.sr/3BgiB2x" (id 4) (at 57.15 121.666 0)
+      (effects (font (size 1.27 1.27)) hide)
+    )
+    (property "FootprintPurchaseUrl" "https://mou.sr/3DAlE8i" (id 5) (at 57.15 121.666 0)
+      (effects (font (size 1.27 1.27)) hide)
+    )
     (pin "1")
     (pin "2")
@@
       (effects (font (size 1.27 1.27)) hide)
     )
-    (property "Purchase" "https://mou.sr/3BzZZfc" (id 4) (at 39.37 52.578 0)
+    (property "ComponentPurchaseUrl" "https://mou.sr/3BzZZfc" (id 4) (at 39.37 52.578 0)
+      (effects (font (size 1.27 1.27)) hide)
+    )
+    (property "FootprintPurchaseUrl" "https://mou.sr/3xt2Q7o" (id 5) (at 39.37 52.578 0)
       (effects (font (size 1.27 1.27)) hide)
     )
@@
       (effects (font (size 1.27 1.27)) hide)
     )
+    (property "ComponentPurchaseUrl" "https://mou.sr/3BgiB2x" (id 4) (at 57.15 121.666 0)
+      (effects (font (size 1.27 1.27)) hide)
+    )
+    (property "FootprintPurchaseUrl" "https://mou.sr/3DAlE8i" (id 5) (at 57.15 121.666 0)
+      (effects (font (size 1.27 1.27)) hide)
+    )
