File: hardware/kicad/6502/vertical.kicad_sch (KiCad schematic)
At the start: 5 parts, among them U11 74LS161, U12 GAL16V8, U13 74HC00, U20 74LS161, U21 74LS161

Commit message: Finalized revision 1.2.
Changed lines of the file:
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@@
+    (stroke (width 0) (type default) (color 0 0 0 0))
+  )
+  (wire (pts (xy 21.59 55.372) (xy 23.876 55.372))
     (stroke (width 0) (type default) (color 0 0 0 0))
   )
@@
     (stroke (width 0) (type default) (color 0 0 0 0))
   )
+  (wire (pts (xy 83.312 55.372) (xy 85.852 55.372))
+    (stroke (width 0) (type default) (color 0 0 0 0))
+  )
   (wire (pts (xy 73.66 119.888) (xy 94.742 130.048))
     (stroke (width 0) (type default) (color 0 0 0 0))
@@
   )
   (wire (pts (xy 115.824 130.048) (xy 115.824 127.254))
+    (stroke (width 0) (type default) (color 0 0 0 0))
+  )
+  (wire (pts (xy 145.796 54.61) (xy 147.574 54.61))
     (stroke (width 0) (type default) (color 0 0 0 0))
   )
@@
     (pin "14")
     (pin "7")
+  )
+  (symbol (lib_id "power:VCC") (at 83.312 55.372 90) (unit 1)
+    (in_bom yes) (on_board yes)
+    (property "Reference" "#PWR0162" (id 0) (at 87.122 55.372 0)
+      (effects (font (size 1.27 1.27)) hide)
+    )
+    (property "Value" "VCC" (id 1) (at 78.232 55.372 90))
+    (property "Footprint" "" (id 2) (at 83.312 55.372 0)
+      (effects (font (size 1.27 1.27)) hide)
+    )
+    (property "Datasheet" "" (id 3) (at 83.312 55.372 0)
+      (effects (font (size 1.27 1.27)) hide)
+    )
+    (pin "1")
   )
   (symbol (lib_id "power:GND") (at 101.346 74.422 0) (unit 1)
@@
     (pin "1")
   )
-  (symbol (lib_id "power:VCC") (at 147.574 54.61 90) (unit 1)
-    (in_bom yes) (on_board yes)
-    (property "Reference" "#PWR052" (id 0) (at 151.384 54.61 0)
-      (effects (font (size 1.27 1.27)) hide)
-    )
-    (property "Value" "VCC" (id 1) (at 142.494 54.61 90))
-    (property "Footprint" "" (id 2) (at 147.574 54.61 0)
-      (effects (font (size 1.27 1.27)) hide)
-    )
-    (property "Datasheet" "" (id 3) (at 147.574 54.61 0)
+  (symbol (lib_id "power:VCC") (at 21.59 55.372 90) (unit 1)
+    (in_bom yes) (on_board yes)
+    (property "Reference" "#PWR0163" (id 0) (at 25.4 55.372 0)
+      (effects (font (size 1.27 1.27)) hide)
+    )
+    (property "Value" "VCC" (id 1) (at 16.51 55.372 90))
+    (property "Footprint" "" (id 2) (at 21.59 55.372 0)
+      (effects (font (size 1.27 1.27)) hide)
+    )
+    (property "Datasheet" "" (id 3) (at 21.59 55.372 0)
       (effects (font (size 1.27 1.27)) hide)
     )
@@
     (pin "7")
   )
-  (symbol (lib_id "power:VCC") (at 85.852 55.372 90) (unit 1)
-    (in_bom yes) (on_board yes)
-    (property "Reference" "#PWR049" (id 0) (at 89.662 55.372 0)
-      (effects (font (size 1.27 1.27)) hide)
-    )
-    (property "Value" "VCC" (id 1) (at 80.772 55.372 90))
-    (property "Footprint" "" (id 2) (at 85.852 55.372 0)
-      (effects (font (size 1.27 1.27)) hide)
-    )
-    (property "Datasheet" "" (id 3) (at 85.852 55.372 0)
-      (effects (font (size 1.27 1.27)) hide)
-    )
-    (pin "1")
-  )
-  (symbol (lib_id "power:VCC") (at 23.876 55.372 90) (unit 1)
-    (in_bom yes) (on_board yes)
-    (property "Reference" "#PWR044" (id 0) (at 27.686 55.372 0)
-      (effects (font (size 1.27 1.27)) hide)
-    )
-    (property "Value" "VCC" (id 1) (at 18.796 55.372 90))
-    (property "Footprint" "" (id 2) (at 23.876 55.372 0)
-      (effects (font (size 1.27 1.27)) hide)
-    )
-    (property "Datasheet" "" (id 3) (at 23.876 55.372 0)
-      (effects (font (size 1.27 1.27)) hide)
-    )
+  (symbol (lib_id "power:VCC") (at 145.796 54.61 90) (unit 1)
+    (in_bom yes) (on_board yes)
+    (property "Reference" "#PWR0161" (id 0) (at 149.606 54.61 0)
+      (effects (font (size 1.27 1.27)) hide)
+    )
+    (property "Value" "VCC" (id 1) (at 140.716 54.61 90))
+    (property "Footprint" "" (id 2) (at 145.796 54.61 0)
+      (effects (font (size 1.27 1.27)) hide)
+    )
+    (property "Datasheet" "" (id 3) (at 145.796 54.61 0)
+      (effects (font (size 1.27 1.27)) hide)
+    )

Commit message: BOM updates.
Parts:
- U11, U20: ComponentPurchaseUrl (none) -> https://mou.sr/3BzZZfc; FootprintPurchaseUrl (none) -> https://mou.sr/3xt2Q7o; Purchase https://mou.sr/3BzZZfc -> (none)
- U12: ComponentPurchaseUrl (none) -> https://mou.sr/3qwJien; FootprintPurchaseUrl (none) -> https://mou.sr/3defX5i; Purchase https://mou.sr/3qwJien -> (none)
- U13: ComponentPurchaseUrl (none) -> https://mou.sr/3BgiB2x; FootprintPurchaseUrl (none) -> https://mou.sr/3DAlE8i
- U21: ComponentPurchaseUrl (none) -> https://mou.sr/3BzZZfc; FootprintPuchaseUrl (none) -> https://mou.sr/3xt2Q7o; Purchase https://mou.sr/3BzZZfc -> (none)
Changed lines of the file:
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@@
+      (effects (font (size 1.27 1.27)) hide)
+    )
+    (property "ComponentPurchaseUrl" "https://mou.sr/3BgiB2x" (id 4) (at 49.276 120.396 0)
+      (effects (font (size 1.27 1.27)) hide)
+    )
+    (property "FootprintPurchaseUrl" "https://mou.sr/3DAlE8i" (id 5) (at 49.276 120.396 0)
       (effects (font (size 1.27 1.27)) hide)
     )
@@
       (effects (font (size 1.27 1.27)) hide)
     )
+    (property "ComponentPurchaseUrl" "https://mou.sr/3BgiB2x" (id 4) (at 49.276 120.396 0)
+      (effects (font (size 1.27 1.27)) hide)
+    )
+    (property "FootprintPurchaseUrl" "https://mou.sr/3DAlE8i" (id 5) (at 49.276 120.396 0)
+      (effects (font (size 1.27 1.27)) hide)
+    )
     (pin "1")
     (pin "2")
@@
       (effects (font (size 1.27 1.27)) hide)
     )
-    (property "Purchase" "https://mou.sr/3BzZZfc" (id 4) (at 163.068 53.34 0)
+    (property "ComponentPurchaseUrl" "https://mou.sr/3BzZZfc" (id 4) (at 163.068 53.34 0)
+      (effects (font (size 1.27 1.27)) hide)
+    )
+    (property "FootprintPuchaseUrl" "https://mou.sr/3xt2Q7o" (id 5) (at 163.068 53.34 0)
       (effects (font (size 1.27 1.27)) hide)
     )
@@
       (effects (font (size 1.27 1.27)) hide)
     )
+    (property "ComponentPurchaseUrl" "https://mou.sr/3BgiB2x" (id 4) (at 49.276 120.396 0)
+      (effects (font (size 1.27 1.27)) hide)
+    )
+    (property "FootprintPurchaseUrl" "https://mou.sr/3DAlE8i" (id 5) (at 49.276 120.396 0)
+      (effects (font (size 1.27 1.27)) hide)
+    )
     (pin "1")
     (pin "2")
@@
       (effects (font (size 1.27 1.27)) hide)
     )
-    (property "Purchase" "https://mou.sr/3BzZZfc" (id 4) (at 101.346 54.102 0)
+    (property "ComponentPurchaseUrl" "https://mou.sr/3BzZZfc" (id 4) (at 101.346 54.102 0)
+      (effects (font (size 1.27 1.27)) hide)
+    )
+    (property "FootprintPurchaseUrl" "https://mou.sr/3xt2Q7o" (id 5) (at 101.346 54.102 0)
       (effects (font (size 1.27 1.27)) hide)
     )
@@
       (effects (font (size 1.27 1.27)) hide)
     )
+    (property "ComponentPurchaseUrl" "https://mou.sr/3BgiB2x" (id 4) (at 49.276 120.396 0)
+      (effects (font (size 1.27 1.27)) hide)
+    )
+    (property "FootprintPurchaseUrl" "https://mou.sr/3DAlE8i" (id 5) (at 49.276 120.396 0)
+      (effects (font (size 1.27 1.27)) hide)
+    )
     (pin "1")
     (pin "2")
@@
       (effects (font (size 1.27 1.27)) hide)
     )
+    (property "ComponentPurchaseUrl" "https://mou.sr/3BgiB2x" (id 4) (at 49.276 120.396 0)
+      (effects (font (size 1.27 1.27)) hide)
+    )
+    (property "FootprintPurchaseUrl" "https://mou.sr/3DAlE8i" (id 5) (at 49.276 120.396 0)
+      (effects (font (size 1.27 1.27)) hide)
+    )
     (pin "1")
     (pin "2")
@@
       (effects (font (size 1.27 1.27)) hide)
     )
-    (property "Purchase" "https://mou.sr/3BzZZfc" (id 4) (at 39.37 52.832 0)
+    (property "ComponentPurchaseUrl" "https://mou.sr/3BzZZfc" (id 4) (at 39.37 52.832 0)
+      (effects (font (size 1.27 1.27)) hide)
+    )
+    (property "FootprintPurchaseUrl" "https://mou.sr/3xt2Q7o" (id 5) (at 39.37 52.832 0)
       (effects (font (size 1.27 1.27)) hide)
     )
@@
       (effects (font (size 1.27 1.27)) hide)
     )
-    (property "Purchase" "https://mou.sr/3qwJien" (id 4) (at 252.222 49.784 0)
-      (effects (font (size 1.27 1.27)) hide)
-    )
+    (property "ComponentPurchaseUrl" "https://mou.sr/3qwJien" (id 4) (at 252.222 49.784 0)
+      (effects (font (size 1.27 1.27)) hide)
+    )
+    (property "FootprintPurchaseUrl" "https://mou.sr/3defX5i" (id 5) (at 252.222 49.784 0)
+      (effects (font (size 1.27 1.27)) hide)
+    )
