File: hardware/kicad/6502/6502.kicad_sch (KiCad schematic)
At the start: 34 parts, among them J1 Barrel_Jack, J2 Bus_Header, J3 VIA_Header, SW1 SW_Push, SW2 SW_Push, SW3 SW_Push, SW4 SW_Push, SW5 SW_Push, U1 L7805, U2 W65C02SxP, U3 28C256, U4 HM62256BLP, U5 W65C22SxP, U6 74LS00, U7 74LS00, X1 TFT680

Commit message: End of day 8/24.
Parts:
- R1, R2, R3, R4, R5, R6: footprint Resistor_THT:R_Axial_Power_L25.0mm_W9.0mm_P10.16mm_Vertical -> Resistor_THT:R_Axial_DIN0207_L6.3mm_D2.5mm_P10.16mm_Horizontal
- U1: footprint Package_TO_SOT_THT:TO-220-5_Horizontal_TabDown -> Package_TO_SOT_THT:TO-220-3_Horizontal_TabDown
- U3, U4: footprint Package_DIP:DIP-28_W15.24mm -> Package_DIP:DIP-28_W15.24mm_Socket
- U5: footprint Package_DIP:DIP-42_W15.24mm -> Package_DIP:DIP-40_W15.24mm_Socket
Changed lines of the file:
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@@
+    (effects (font (size 1.27 1.27)) (justify left bottom))
+  )
+  (text "LEFT" (at 233.68 78.74 90)
     (effects (font (size 1.27 1.27)) (justify left bottom))
   )
@@
       (effects (font (size 1.27 1.27)) (justify left))
     )
-    (property "Footprint" "Resistor_THT:R_Axial_Power_L25.0mm_W9.0mm_P10.16mm_Vertical" (id 2) (at 261.62 62.23 90)
+    (property "Footprint" "Resistor_THT:R_Axial_DIN0207_L6.3mm_D2.5mm_P10.16mm_Horizontal" (id 2) (at 261.62 62.23 90)
       (effects (font (size 1.27 1.27)) hide)
     )
@@
     (property "Reference" "U1" (id 0) (at 59.944 165.1 0))
     (property "Value" "L7805" (id 1) (at 59.944 167.64 0))
-    (property "Footprint" "Package_TO_SOT_THT:TO-220-5_Horizontal_TabDown" (id 2) (at 60.579 176.53 0)
+    (property "Footprint" "Package_TO_SOT_THT:TO-220-3_Horizontal_TabDown" (id 2) (at 60.579 176.53 0)
       (effects (font (size 1.27 1.27) italic) (justify left) hide)
     )
@@
       (effects (font (size 1.27 1.27)) (justify left))
     )
-    (property "Footprint" "Resistor_THT:R_Axial_Power_L25.0mm_W9.0mm_P10.16mm_Vertical" (id 2) (at 249.936 62.23 90)
+    (property "Footprint" "Resistor_THT:R_Axial_DIN0207_L6.3mm_D2.5mm_P10.16mm_Horizontal" (id 2) (at 249.936 62.23 90)
       (effects (font (size 1.27 1.27)) hide)
     )
@@
       (effects (font (size 1.27 1.27)) (justify left))
     )
-    (property "Footprint" "Resistor_THT:R_Axial_Power_L25.0mm_W9.0mm_P10.16mm_Vertical" (id 2) (at 238.252 62.23 90)
+    (property "Footprint" "Resistor_THT:R_Axial_DIN0207_L6.3mm_D2.5mm_P10.16mm_Horizontal" (id 2) (at 238.252 62.23 90)
       (effects (font (size 1.27 1.27)) hide)
     )
@@
       (effects (font (size 1.27 1.27)) (justify left))
     )
-    (property "Footprint" "Resistor_THT:R_Axial_Power_L25.0mm_W9.0mm_P10.16mm_Vertical" (id 2) (at 86.36 185.166 90)
+    (property "Footprint" "Resistor_THT:R_Axial_DIN0207_L6.3mm_D2.5mm_P10.16mm_Horizontal" (id 2) (at 86.36 185.166 90)
       (effects (font (size 1.27 1.27)) hide)
     )
@@
       (effects (font (size 1.27 1.27)) (justify left))
     )
-    (property "Footprint" "Package_DIP:DIP-28_W15.24mm" (id 2) (at 94.234 51.562 0)
+    (property "Footprint" "Package_DIP:DIP-28_W15.24mm_Socket" (id 2) (at 94.234 51.562 0)
       (effects (font (size 1.27 1.27)) hide)
     )
@@
       (effects (font (size 1.27 1.27)) (justify left))
     )
-    (property "Footprint" "Resistor_THT:R_Axial_Power_L25.0mm_W9.0mm_P10.16mm_Vertical" (id 2) (at 148.082 176.276 90)
+    (property "Footprint" "Resistor_THT:R_Axial_DIN0207_L6.3mm_D2.5mm_P10.16mm_Horizontal" (id 2) (at 148.082 176.276 90)
       (effects (font (size 1.27 1.27)) hide)
     )
@@
       (effects (font (size 1.27 1.27)) (justify left))
     )
-    (property "Footprint" "Resistor_THT:R_Axial_Power_L25.0mm_W9.0mm_P10.16mm_Vertical" (id 2) (at 273.558 62.23 90)
+    (property "Footprint" "Resistor_THT:R_Axial_DIN0207_L6.3mm_D2.5mm_P10.16mm_Horizontal" (id 2) (at 273.558 62.23 90)
       (effects (font (size 1.27 1.27)) hide)
     )
@@
       (effects (font (size 1.27 1.27) bold italic) (justify left))
     )
-    (property "Footprint" "Package_DIP:DIP-42_W15.24mm" (id 2) (at 200.914 54.61 0)
+    (property "Footprint" "Package_DIP:DIP-40_W15.24mm_Socket" (id 2) (at 200.914 54.61 0)
       (effects (font (size 1.27 1.27)) hide)
     )
@@
       (effects (font (size 1.27 1.27)) (justify left))
     )
-    (property "Footprint" "Package_DIP:DIP-28_W15.24mm" (id 2) (at 145.288 49.022 0)
+    (property "Footprint" "Package_DIP:DIP-28_W15.24mm_Socket" (id 2) (at 145.288 49.022 0)
       (effects (font (size 1.27 1.27)) hide)
     )
@@
     )
     (path "/53c690db-9b8f-41fe-b1d0-752e26383d89"
-      (reference "R1") (unit 1) (value "1k") (footprint "Resistor_THT:R_Axial_Power_L25.0mm_W9.0mm_P10.16mm_Vertical")
+      (reference "R1") (unit 1) (value "1k") (footprint "Resistor_THT:R_Axial_DIN0207_L6.3mm_D2.5mm_P10.16mm_Horizontal")
     )
     (path "/724faffe-d81a-430b-b36a-214d0825f121"
-      (reference "R2") (unit 1) (value "1k") (footprint "Resistor_THT:R_Axial_Power_L25.0mm_W9.0mm_P10.16mm_Vertical")
+      (reference "R2") (unit 1) (value "1k") (footprint "Resistor_THT:R_Axial_DIN0207_L6.3mm_D2.5mm_P10.16mm_Horizontal")
     )
     (path "/3f57b748-9184-4759-9ec5-f88367939c40"
-      (reference "R3") (unit 1) (value "1k") (footprint "Resistor_THT:R_Axial_Power_L25.0mm_W9.0mm_P10.16mm_Vertical")
+      (reference "R3") (unit 1) (value "1k") (footprint "Resistor_THT:R_Axial_DIN0207_L6.3mm_D2.5mm_P10.16mm_Horizontal")
     )
     (path "/121d86b8-086e-4e4a-9150-3db8272ed652"
-      (reference "R4") (unit 1) (value "1k") (footprint "Resistor_THT:R_Axial_Power_L25.0mm_W9.0mm_P10.16mm_Vertical")
+      (reference "R4") (unit 1) (value "1k") (footprint "Resistor_THT:R_Axial_DIN0207_L6.3mm_D2.5mm_P10.16mm_Horizontal")
     )
     (path "/030ba778-d589-4227-a2c2-e8bb8295a663"
-      (reference "R5") (unit 1) (value "1k") (footprint "Resistor_THT:R_Axial_Power_L25.0mm_W9.0mm_P10.16mm_Vertical")
+      (reference "R5") (unit 1) (value "1k") (footprint "Resistor_THT:R_Axial_DIN0207_L6.3mm_D2.5mm_P10.16mm_Horizontal")
     )
     (path "/b4dff0cd-b56f-4427-952d-8b3b8fe93d87"
-      (reference "R6") (unit 1) (value "1k") (footprint "Resistor_THT:R_Axial_Power_L25.0mm_W9.0mm_P10.16mm_Vertical")
+      (reference "R6") (unit 1) (value "1k") (footprint "Resistor_THT:R_Axial_DIN0207_L6.3mm_D2.5mm_P10.16mm_Horizontal")
     )
     (path "/05399a96-ac24-42d3-8633-ebf1b2c62140"
@@
     )
     (path "/0e871afd-1767-4694-b981-756f16069fdd"
-      (reference "U1") (unit 1) (value "L7805") (footprint "Package_TO_SOT_THT:TO-220-5_Horizontal_TabDown")
+      (reference "U1") (unit 1) (value "L7805") (footprint "Package_TO_SOT_THT:TO-220-3_Horizontal_TabDown")
     )
     (path "/8dcfd59b-a304-4f6c-99aa-4b3035708ab3"
@@
     )
     (path "/57d520a1-d8d6-4532-b8f4-05b97dc3bc7b"
-      (reference "U3") (unit 1) (value "28C256") (footprint "Package_DIP:DIP-28_W15.24mm")
+      (reference "U3") (unit 1) (value "28C256") (footprint "Package_DIP:DIP-28_W15.24mm_Socket")
     )
     (path "/e6e3381a-a81d-42c3-a4d5-fcaba8baaad6"
-      (reference "U4") (unit 1) (value "HM62256BLP") (footprint "Package_DIP:DIP-28_W15.24mm")
+      (reference "U4") (unit 1) (value "HM62256BLP") (footprint "Package_DIP:DIP-28_W15.24mm_Socket")
     )
     (path "/dd739fba-aa49-4b3c-a169-28c668fbec5c"
-      (reference "U5") (unit 1) (value "W65C22SxP") (footprint "Package_DIP:DIP-42_W15.24mm")
+      (reference "U5") (unit 1) (value "W65C22SxP") (footprint "Package_DIP:DIP-40_W15.24mm_Socket")
     )
     (path "/0697e705-14c7-43dc-ac7c-e4b76905cb47"

Commit message: Corrected some minor rev 1.0 issues.
Connections:
- net GND: now also J3.1 (Pin_1); no longer J3.2 (Pin_2)
- net VCC: now also J3.2 (Pin_2); no longer J3.1 (Pin_1), RV1.3
- no-connect marks 10 -> 11
Changed lines of the file:
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@@
   (title_block
     (title "6502 Prototype")
-    (date "8/23/2022")
-    (rev "1.0")
+    (date "9/2/2022")
+    (rev "1.1")
     (company "Korey Bliss")
     (comment 1 "https://github.com/kblissExternal/6502")
@@
   (no_connect (at 19.304 39.878))
   (no_connect (at 19.304 42.418))
+  (no_connect (at 239.268 111.76))
   (no_connect (at 276.098 151.384))
   (no_connect (at 276.098 148.844))
@@
     (stroke (width 0) (type default) (color 0 0 0 0))
   )
-  (wire (pts (xy 232.41 125.984) (xy 235.458 125.984))
-    (stroke (width 0) (type default) (color 0 0 0 0))
-  )
   (wire (pts (xy 81.534 135.636) (xy 87.122 135.636))
     (stroke (width 0) (type default) (color 0 0 0 0))
@@
     (stroke (width 0) (type default) (color 0 0 0 0))
   )
-  (wire (pts (xy 232.156 128.524) (xy 235.458 128.524))
-    (stroke (width 0) (type default) (color 0 0 0 0))
-  )
   (wire (pts (xy 260.604 69.342) (xy 260.604 65.786))
     (stroke (width 0) (type default) (color 0 0 0 0))
@@
     (pin "1")
   )
-  (symbol (lib_id "power:VCC") (at 232.41 125.984 90) (unit 1)
+  (symbol (lib_id "power:VCC") (at 235.458 128.524 90) (unit 1)
     (in_bom yes) (on_board yes)
-    (property "Reference" "#PWR030" (id 0) (at 236.22 125.984 0)
+    (property "Reference" "#PWR030" (id 0) (at 239.268 128.524 0)
       (effects (font (size 1.27 1.27)) hide)
     )
-    (property "Value" "VCC" (id 1) (at 227.33 125.984 90))
-    (property "Footprint" "" (id 2) (at 232.41 125.984 0)
+    (property "Value" "VCC" (id 1) (at 230.378 128.524 90))
+    (property "Footprint" "" (id 2) (at 235.458 128.524 0)
       (effects (font (size 1.27 1.27)) hide)
     )
-    (property "Datasheet" "" (id 3) (at 232.41 125.984 0)
+    (property "Datasheet" "" (id 3) (at 235.458 128.524 0)
       (effects (font (size 1.27 1.27)) hide)
     )
@@
     (pin "1")
   )
-  (symbol (lib_id "power:GND") (at 232.156 128.524 270) (unit 1)
+  (symbol (lib_id "power:GND") (at 235.458 125.984 270) (unit 1)
     (in_bom yes) (on_board yes)
-    (property "Reference" "#PWR028" (id 0) (at 225.806 128.524 0)
+    (property "Reference" "#PWR028" (id 0) (at 229.108 125.984 0)
       (effects (font (size 1.27 1.27)) hide)
     )
-    (property "Value" "GND" (id 1) (at 227.33 128.524 90))
-    (property "Footprint" "" (id 2) (at 232.156 128.524 0)
+    (property "Value" "GND" (id 1) (at 230.632 125.984 90))
+    (property "Footprint" "" (id 2) (at 235.458 125.984 0)
       (effects (font (size 1.27 1.27)) hide)
     )
-    (property "Datasheet" "" (id 3) (at 232.156 128.524 0)
+    (property "Datasheet" "" (id 3) (at 235.458 125.984 0)
       (effects (font (size 1.27 1.27)) hide)
     )
@@
     (pin "9")
   )
-  (symbol (lib_id "power:VCC") (at 239.268 111.76 270) (unit 1)
-    (in_bom yes) (on_board yes)
-    (property "Reference" "#PWR032" (id 0) (at 235.458 111.76 0)
-      (effects (font (size 1.27 1.27)) hide)
-    )
-    (property "Value" "VCC" (id 1) (at 244.348 111.76 0))
-    (property "Footprint" "" (id 2) (at 239.268 111.76 0)
-      (effects (font (size 1.27 1.27)) hide)
-    )
-    (property "Datasheet" "" (id 3) (at 239.268 111.76 0)
-      (effects (font (size 1.27 1.27)) hide)
-    )
-    (pin "1")
-  )
   (symbol (lib_id "74xx:74LS00") (at 55.88 136.906 0) (unit 2)
     (in_bom yes) (on_board yes) (fields_autoplaced)
@@
       (reference "#PWR031") (unit 1) (value "VCC") (footprint "")
     )
-    (path "/e74dd862-6e25-4aab-84c8-2ad8ae153cdf"
-      (reference "#PWR032") (unit 1) (value "VCC") (footprint "")
-    )
     (path "/1f641064-e1a7-45c2-a724-de76ab5af39e"

Commit message: Update to Revision 1.1 (primarily adding 6551).
Parts:
- added C10: 33pF, Capacitor_THT:C_Disc_D5.0mm_W2.5mm_P5.00mm, symbol Device:C
- added C11, C12: 0.1µF, Capacitor_THT:C_Disc_D5.0mm_W2.5mm_P2.50mm, symbol Device:C
- added J4: UART_Header, Connector_PinSocket_2.54mm:PinSocket_1x06_P2.54mm_Vertical, symbol Connector:Conn_01x06_Female
- added J5: VIA_Header, Connector_PinSocket_2.54mm:PinSocket_1x16_P2.54mm_Vertical, symbol Connector:Conn_01x16_Female
- added U8: W65C51NxP, Package_DIP:DIP-28_W15.24mm_Socket, symbol 65xx:W65C51NxP
- added U9: 74LS00, Package_DIP:DIP-14_W7.62mm_Socket, symbol 74xx:74LS00
- added X2: TFT680, Oscillator:Oscillator_DIP-14, symbol Oscillator:TFT680
- J3: value VIA_Header -> LCD_Header
Connections:
- net A0: now also U8.13 (RS0)
- net A1: now also U8.14 (RS1)
- net A13: now also U9.1, U9.2
- net D0: now also U8.18 (D0)
- net D1: now also U8.19 (D1)
- net D2: now also U8.20 (D2)
- net D3: now also U8.21 (D3)
- net D4: now also U8.22 (D4)
- net D5: now also U8.23 (D5)
- net D6: now also U8.24 (D6)
- net D7: now also U8.25 (D7)
- net GND: now also C10.2, C11.1, C12.1, J4.1 (Pin_1), J4.6 (Pin_6), U8.1 (VSS), U8.11 (~{DTR}), U8.16 (~{DCD}), U8.17 (~{DSR}), U8.9 (~{CTS}), U9.10, U9.12, U9.13, U9.4, U9.5, U9.7 (GND), U9.9, X2.7 (GND)
- net PA0: now also J5.1 (Pin_1)
- net PA1: now also J5.2 (Pin_2)
- net PA2: now also J5.3 (Pin_3)
- net PA3: now also J5.4 (Pin_4)
- net PA4: now also J5.5 (Pin_5)
- net PA5: now also J5.6 (Pin_6)
- net PA6: now also J5.7 (Pin_7)
- net PA7: now also J5.8 (Pin_8)
- net PB0: now also J5.9 (Pin_9)
- net PB1: now also J5.10 (Pin_10)
- net PB2: now also J5.11 (Pin_11)
- net PB3: now also J5.12 (Pin_12)
- net PB4: now also J5.13 (Pin_13)
- net PB5: now also J5.14 (Pin_14)
- net PB6: now also J5.15 (Pin_15)
- net PB7: now also J5.16 (Pin_16)
- net PHI2: now also U7.9, U8.27 (ϕ2)
- net VCC: now also C11.2, C12.2, U8.15 (VCC), U9.14 (VCC), X2.14 (Vcc)
- net ~{IRQ}: now also U8.26 (~{IRQ})
- net ~{PHI2}: no longer U7.9
- net ~{RES}: now also U8.4 (~{RES})
- net ~{RW}: now also U8.28 (R/~{W})
- net ~{VIACS2}: now also U8.3 (~{CS1})
- new net PHI3: C10.1, U8.6 (XTLI), X2.8 (OUT)
- new net UART_RX: J4.3 (Pin_3), U8.12 (RxD)
- new net UART_TX: J4.2 (Pin_2), U8.10 (TxD)
- new net ~{ACIACS}: U8.2 (CS0), U9.3
- new net ~{UART_RTS}: J4.5 (Pin_5), U8.8 (~{RTS})
- no-connect marks 11 -> 18
Other:
- note added: "65xx ICs"
- note added: "Baud Rate Clock"
- moved on the sheet: C1, C2, C3, C4, C5, C6, C7, C8, C9, D1, D2, J1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

Commit message: Added VGA testing components.
Parts:
- removed C1: 1µF, Capacitor_THT:C_Radial_D4.0mm_H5.0mm_P1.50mm, symbol Device:C_Polarized
- removed C7: 0.1µF, Capacitor_THT:C_Disc_D5.0mm_W2.5mm_P2.50mm, symbol Device:C
- removed U1: L7805, Package_TO_SOT_THT:TO-220-3_Horizontal_TabDown, symbol Regulator_Linear:L7805
- removed U6, U7, U9: 74LS00, Package_DIP:DIP-14_W7.62mm_Socket, symbol 74xx:74LS00
- added J7: GAL_Header, Connector_PinSocket_2.54mm:PinSocket_1x16_P2.54mm_Vertical, symbol Connector:Conn_01x16_Female
- added SW8: SW_SPDT, Switch:SW_THT_DPDT, symbol Switch:SW_SPDT
- added U1: GAL16V8, Package_DIP:DIP-20_W7.62mm_Socket, symbol Logic_Programmable:GAL16V8
- C1: renamed from C2; value 0.1µF -> 1µF; footprint Capacitor_THT:C_Disc_D5.0mm_W2.5mm_P2.50mm -> Capacitor_THT:C_Radial_D4.0mm_H5.0mm_P1.50mm; Purchase (none) -> https://mou.sr/3RYvaGw
- C2: renamed from C8; Purchase (none) -> https://mou.sr/3L92t7l
- C3: renamed from C9; Purchase (none) -> https://mou.sr/3L92t7l
- C4: renamed from C3; Purchase (none) -> https://mou.sr/3L92t7l
- C5: renamed from C4; Purchase (none) -> https://mou.sr/3L92t7l
- C6: renamed from C5; Purchase (none) -> https://mou.sr/3L92t7l
- C7: renamed from C6; Purchase (none) -> https://mou.sr/3L92t7l
- C8: renamed from C11; Purchase (none) -> https://mou.sr/3L92t7l
- C9: renamed from C12; Purchase (none) -> https://mou.sr/3L92t7l
- D1: Purchase (none) -> https://mou.sr/3BAfBiO
- J1: Purchase (none) -> https://mou.sr/3eDGF7P
- R1, R2, R3: Purchase (none) -> https://mou.sr/3xhN8M1
- SW1, SW2, SW3, SW4, SW5: Purchase (none) -> https://mou.sr/3eIzPy2
- U2: Purchase (none) -> https://mou.sr/3Dkbt7V
- U3: Purchase (none) -> https://mou.sr/3RUXglV
- U4: Purchase (none) -> https://mou.sr/3qzRFG5
- U5: Purchase (none) -> https://mou.sr/3RH02f0
- U8: Purchase (none) -> https://mou.sr/3B4roEC
- X1: Purchase (none) -> https://mou.sr/3BddYWK
- X2: Purchase (none) -> https://mou.sr/3RDGI29
- renumbered C10 to C11
Connections:
- net PHI3 is gone; now on net PHI2: C11.1, U8.6 (XTLI), X2.8 (OUT)
- net A12: now also U1.1 (I1/CLK)
- net A13: now also U1.2 (I2); no longer U5.24 (CS1)
- net A14: now also U1.3 (I3); no longer U4.22 (~{OE})
- net A15: now also U1.4 (I4)
- net GND: now also J7.15 (Pin_15), J7.16 (Pin_16), U1.10 (GND)
- net PHI2: no longer J2.34 (Pin_34), J2.35 (Pin_35), U2.37 (ϕ0), U5.25 (ϕ2), U8.27 (ϕ2)
- net VCC: now also D1.1 (K), U5.24 (CS1), U8.2 (CS0), J7.14 (Pin_14), U1.20 (VCC)
- net ~{ACIACS}: now also U8.3 (~{CS1}), U1.14 (IO6); no longer U8.2 (CS0)
- net ~{RAMCS}: now also U1.18 (IO2)
- net ~{ROMCS}: now also U1.19 (IO1)
- net ~{HBLANK}: now reaches J2.24 (Pin_24)
- net ~{VBLANK}: now reaches J2.26 (Pin_26)
- net ~{HSYNC}: now reaches J2.28 (Pin_28)
- net ~{VSYNC}: now reaches J2.30 (Pin_30)
- net at D1.2 (A): now also SW8.1 (A); no longer J1.1
- net RDY renamed ~{DMA}
- net ~{DMA}: now also U1.5 (I5)
- net ~{PHI2} renamed ~{CPU_CLOCK}
- net ~{CPU_CLOCK}: now also U1.16 (IO4)
- net ~{VIACS2} renamed ~{VIACS}
- net ~{VIACS}: now also U1.15 (IO5); no longer U8.3 (~{CS1})
- new net: J1.1, SW8.2 (B)
- new net CPU_CLOCK: J2.34 (Pin_34), J2.35 (Pin_35), U1.6 (I6), U2.37 (ϕ0), U5.25 (ϕ2), U8.27 (ϕ2)
- new net GAL0_I0: J7.1 (Pin_1), U1.7 (I7)
- new net GAL0_I1: J7.2 (Pin_2), U1.8 (I8)
- new net GAL0_I2: J7.3 (Pin_3), U1.9 (I9)
- new net GAL0_I3: J7.4 (Pin_4), U1.11 (I10/~{OE})
- new net GAL0_O0: J7.8 (Pin_8), U1.13 (IO7)
- new net GAL0_O1: J7.9 (Pin_9), U1.12 (IO8)
- new net GAL3_I0: J7.5 (Pin_5)
- new net GAL3_I1: J7.6 (Pin_6)
- new net GAL3_I2: J7.7 (Pin_7)
- new net GAL3_O0: J7.10 (Pin_10)
- new net GAL3_O1: J7.11 (Pin_11)
- new net GAL3_O2: J7.12 (Pin_12)
- new net GAL3_O3: J7.13 (Pin_13)
- new net ~{RAMOE}: U1.17 (I03), U4.22 (~{OE})
- no-connect marks 18 -> 12
Other:
- added sheet VGA (vga.kicad_sch)
- note added: "Control Input"
- note removed: "Button Input"
- moved on the sheet: C1, C11, D1, D2, J1, J2, J3, J4, J5, R1, R2, R3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

Commit message: Finalized revision 1.2.
Connections:
- net A12: now also U1.2 (I2); no longer U1.1 (I1/CLK)
- net A13: now also U1.3 (I3); no longer U1.2 (I2)
- net A14: now also U1.4 (I4); no longer U1.3 (I3)
- net A15: now also U1.5 (I5); no longer U1.4 (I4)
- net CPU_CLOCK: now also U1.1 (I1/CLK); no longer U1.6 (I6)
- net GAL0_O0: now also U1.12 (IO8); no longer U1.13 (IO7)
- net GAL3_O0: now also J7.9 (Pin_9); no longer J7.10 (Pin_10)
- net GAL3_O1: now also J7.10 (Pin_10); no longer J7.11 (Pin_11)
- net GAL3_O2: now also J7.11 (Pin_11); no longer J7.12 (Pin_12)
- net GAL3_O3: now also J7.12 (Pin_12); no longer J7.13 (Pin_13)
- net VCC: now also J7.13 (Pin_13)
- net ~{ACIACS}: now also U1.15 (IO5); no longer U1.14 (IO6)
- net ~{CPU_CLOCK}: now also U1.13 (IO7); no longer U1.16 (IO4)
- net ~{DMA}: now also U1.6 (I6); no longer U1.5 (I5), U2.2 (RDY), U2.36 (BE)
- net ~{VIACS}: now also U1.16 (IO4); no longer U1.15 (IO5)
- removed net GAL0_O1: J7.9 (Pin_9), U1.12 (IO8)
- new net CPU_READY: U1.14 (IO6), U2.2 (RDY), U2.36 (BE)
Other:
- sheet VGA ports: added VGA_CLOCK, ~{H_CLR}; removed none
- moved on the sheet: C1

Commit message: BOM updates.
Parts:
- C1: ComponentPurchaseUrl (none) -> https://mou.sr/3RYvaGw; Purchase https://mou.sr/3RYvaGw -> (none)
- C11: ComponentPurchaseUrl (none) -> https://mou.sr/3Uc47cD
- C2, C3, C4, C5, C6, C7, C8, C9: ComponentPurchaseUrl (none) -> https://mou.sr/3L92t7l; Purchase https://mou.sr/3L92t7l -> (none)
- D1: ComponentPurchaseUrl (none) -> https://mou.sr/3BAfBiO; Purchase https://mou.sr/3BAfBiO -> (none)
- J1: ComponentPurchaseUrl (none) -> https://mou.sr/3eDGF7P; Purchase https://mou.sr/3eDGF7P -> (none)
- J2: ComponentPurchaseUrl (none) -> https://mou.sr/3do1bsG
- J3, J5: ComponentPurchaseUrl (none) -> https://mou.sr/3RRFn7V
- J4: ComponentPurchaseUrl (none) -> https://mou.sr/3BaX7UI
- J7: ComponentPurchaseUrl (none) -> https://mou.sr/3QNGOmm
- R1, R2, R3: ComponentPurchaseUrl (none) -> https://mou.sr/3xhN8M1; Purchase https://mou.sr/3xhN8M1 -> (none)
- RV1: ComponentPurchaseUrl (none) -> https://mou.sr/3S83Aqs
- SW1, SW2, SW3, SW4, SW5: ComponentPurchaseUrl (none) -> https://mou.sr/3eIzPy2; Purchase https://mou.sr/3eIzPy2 -> (none)
- SW8: ComponentPurchaseUrl (none) -> https://mou.sr/3U40nK1; Purchase https://mou.sr/3U40nK1 -> (none)
- U1: ComponentPurchaseUrl (none) -> https://mou.sr/3qwJien; FootprintPurchaseUrl (none) -> https://mou.sr/3defX5i; Purchase https://mou.sr/3qwJien -> (none)
- U2: ComponentPurchaseUrl (none) -> https://mou.sr/3Dkbt7V; FootprintPurchaseUrl (none) -> https://mou.sr/3qH9jaO; Purchase https://mou.sr/3Dkbt7V -> (none)
- U3: ComponentPurchaseUrl (none) -> https://mou.sr/3RUXglV; FootprintPurchaseUrl (none) -> https://mou.sr/3BkyTHw; Purchase https://mou.sr/3RUXglV -> (none)
- U4: ComponentPurchaseUrl (none) -> https://mou.sr/3qzRFG5; FootprintPurchaseUrl (none) -> https://mou.sr/3LexIOA; Purchase https://mou.sr/3qzRFG5 -> (none)
- U5: ComponentPurchaseUrl (none) -> https://mou.sr/3RH02f0; FootprintPurchaseUrl (none) -> https://mou.sr/3qH9jaO; Purchase https://mou.sr/3RH02f0 -> (none)
- U8: ComponentPurchaseUrl (none) -> https://mou.sr/3B4roEC; FootprintPurchaseUrl (none) -> https://mou.sr/3LexIOA; Purchase https://mou.sr/3B4roEC -> (none)
- X1: ComponentPurchaseUrl (none) -> https://mou.sr/3BddYWK; FootprintPurchaseUrl (none) -> https://mou.sr/3DAfghk; Purchase https://mou.sr/3BddYWK -> (none)
- X2: ComponentPurchaseUrl (none) -> https://mou.sr/3RDGI29; Purchase https://mou.sr/3RDGI29 -> (none)
