File: hardware/kicad/6502/vga.kicad_sch (KiCad schematic)
At the start: 35 parts, among them J10 VGA_Data_Header, J6 VGA_Out, J8 VGA_Address_Header, J9 VGA_Clock, SW6 SW_VGA_CLOCK, SW7 DMA_DIP, U14 74HC74, U15 74HC245, U16 74HC245, U17 74HC245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

Commit message: Finalized revision 1.2.
Parts:
- added C10: 0.1µF, Capacitor_THT:C_Disc_D5.0mm_W2.5mm_P2.50mm, symbol Device:C
Connections:
- net GND: now also C10.1
- net VCC: now also C10.2
- net ~{CPU_CLOCK}: now also U9.1 (I1/CLK); no longer U9.3 (I3)
- net ~{HBLANK}: now also U9.2 (I2); no longer U9.1 (I1/CLK)
- net ~{VBLANK}: now also U9.3 (I3); no longer U9.2 (I2)
Other:
- moved on the sheet: C12, C13, C14, C15, C16, C17, C18, C19, C20, C21, C22, C23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

Commit message: BOM updates.
Parts:
- C10, C12, C13, C14, C15, C16, C17, C18, C19, C20, C21, C22, C23: ComponentPurchaseUrl (none) -> https://mou.sr/3L92t7l; Purchase https://mou.sr/3L92t7l -> (none)
- J10: ComponentPurchaseUrl (none) -> https://mou.sr/3Dn1XRw
- J6: ComponentPurchaseUrl (none) -> https://mou.sr/3U9t1cS
- J8: ComponentPurchaseUrl (none) -> https://mou.sr/3do1bsG
- J9: ComponentPurchaseUrl (none) -> https://mou.sr/3UbDc0q
- R10, R12, R8: ComponentPurchaseUrl (none) -> https://mou.sr/3qJ1EZL
- R11, R7, R9: ComponentPurchaseUrl (none) -> https://mou.sr/3qEoBgq
- R13, R14, R15, R16: ComponentPurchaseUrl (none) -> https://mou.sr/3RNFvp2
- SW6: ComponentPurchaseUrl (none) -> https://mou.sr/3U40nK1; Purchase https://mou.sr/3U40nK1 -> (none)
- SW7: ComponentPurchaseUrl (none) -> https://mou.sr/3QRpygp; Purchase https://mou.sr/3QRpygp -> (none)
- U14: ComponentPurchaseUrl (none) -> https://mou.sr/3RKX1tT; FootprintPurchaseUrl (none) -> https://mou.sr/3DAlE8i
- U15, U16, U17: ComponentPurchaseUrl (none) -> https://mou.sr/3U6tr3P; FootprintPurchaseUrl (none) -> https://mou.sr/3defX5i
- U9: ComponentPurchaseUrl (none) -> https://mou.sr/3qwJien; FootprintPurchaseUrl (none) -> https://mou.sr/3defX5i; Purchase https://mou.sr/3qwJien -> (none)
- X3: ComponentPurchaseUrl (none) -> https://mou.sr/3qGWkpK; FootprintPurchaseUrl (none) -> https://mou.sr/3Uf4zXu
- X4: ComponentPurchaseUrl (none) -> https://mou.sr/3RDGI29; FootprintPurchaseUrl (none) -> https://mou.sr/3DAfghk

Commit message: Baseline for VGA functionality.
Connections:
- net GND: no longer J6.9
- net VGA_BLUE: now also J6.3; no longer J6.2
- net VGA_GREEN: now also J6.2; no longer J6.3
- net ~{HSYNC}: now also J6.13; no longer J6.14
- net ~{VSYNC}: now also J6.14; no longer J6.13
- no-connect marks 12 -> 13
Changed lines of the file:
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@@
   (no_connect (at 163.322 191.262))
   (no_connect (at 167.894 102.362))
+  (no_connect (at 148.082 183.642))
   (bus_entry (at 131.572 155.194) (size 2.54 2.54)
     (stroke (width 0) (type default) (color 0 0 0 0))
@@
     (effects (font (size 1.27 1.27)) (justify left bottom))
   )
-  (label "VGA_GREEN" (at 137.414 181.102 0)
+  (label "VGA_BLUE" (at 137.414 181.102 0)
     (effects (font (size 1.27 1.27)) (justify left bottom))
   )
@@
     (effects (font (size 1.27 1.27)) (justify right bottom))
   )
-  (label "VGA_BLUE" (at 137.16 176.022 0)
+  (label "VGA_GREEN" (at 137.16 176.022 0)
     (effects (font (size 1.27 1.27)) (justify left bottom))
   )
@@
     (effects (font (size 1.27 1.27)) (justify left))
   )
-  (hierarchical_label "~{HSYNC}" (shape input) (at 165.862 186.182 0)
+  (hierarchical_label "~{VSYNC}" (shape input) (at 165.862 186.182 0)
     (effects (font (size 1.27 1.27)) (justify left))
   )
@@
     (effects (font (size 1.27 1.27)) (justify left))
   )
-  (hierarchical_label "~{VSYNC}" (shape input) (at 165.862 181.102 0)
+  (hierarchical_label "~{HSYNC}" (shape input) (at 165.862 181.102 0)
     (effects (font (size 1.27 1.27)) (justify left))
   )
@@
     (pin "8")
   )
-  (symbol (lib_id "power:GND") (at 148.082 183.642 270) (unit 1)
-    (in_bom yes) (on_board yes)
-    (property "Reference" "#PWR0111" (id 0) (at 141.732 183.642 0)
-      (effects (font (size 1.27 1.27)) hide)
-    )
-    (property "Value" "GND" (id 1) (at 143.002 183.642 90))
-    (property "Footprint" "" (id 2) (at 148.082 183.642 0)
-      (effects (font (size 1.27 1.27)) hide)
-    )
-    (property "Datasheet" "" (id 3) (at 148.082 183.642 0)
-      (effects (font (size 1.27 1.27)) hide)
-    )
-    (pin "1")
-  )
   (symbol (lib_id "power:VCC") (at 157.48 56.642 90) (unit 1)
